File: bms.kicad_sch (KiCad schematic)
At the start: 64 parts, among them J2 Molex_Pico-Clasp_1x7_Horizont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, J3 Screw_Terminal_01x02, Q13 DMG2301L, Q14 Si1442DH, Q15 CSD17579Q5A, Q16 SiA453EDJ, Q18 2N7002K, Q2 CSD17579Q5A, Q5 DMN2056U, Q8 DMN2056U, Q9 DMN2056U, U1 BQ29410_TSSOP, U4 BQ40Z50RSMT-R2

Commit message: Link footprints and symbols to local lib
Parts:
- C10, C11, C12, C14, C15, C19, C2, C24, C28, C3, C31, C32, C33, C34, C4, C6, C8, C9: symbol Device:C_Small -> pmu_symbols:C_Small
- D1: symbol Diode:BAT54J -> pmu_symbols:BAT54J
- F2: symbol ITV4030_LTF:ITV4030L1412NR -> pmu_symbols:ITV4030L1412NR
- J2: symbol Connector_Generic:Conn_01x08 -> pmu_symbols:Conn_01x08
- J3: symbol Connector:Screw_Terminal_01x02 -> pmu_symbols:Screw_Terminal_01x02
- PTC2, R10, R12, R13, R14, R16, R17, R18, R19, R2, R20, R23, R26, R28, R29, R3, R30, R33, R37, R4, R42, R43, R44, R45, R46, R5, R50, R56, R6, R9: symbol Device:R_Small -> pmu_symbols:R_Small
- Q13: symbol Transistor_FET:DMG2301L -> pmu_symbols:DMG2301L
- Q14: symbol Transistor_FET:Si1442DH -> pmu_symbols:Si1442DH
- Q15, Q2: symbol Transistor_FET:CSD17579Q5A -> pmu_symbols:CSD17579Q5A
- Q16: symbol Transistor_FET:SiA453EDJ -> pmu_symbols:SiA453EDJ
- Q18: symbol Transistor_FET:2N7002K -> pmu_symbols:2N7002K
- Q5, Q8, Q9: symbol Transistor_FET:DMN2056U -> pmu_symbols:DMN2056U
- U1: symbol bq29410_tssop:BQ29410_TSSOP -> pmu_symbols:BQ29410_TSSOP
- U4: symbol BQ40Z50RSMT-R2:BQ40Z50RSMT-R2 -> pmu_symbols:BQ40Z50RSMT-R2
- xx1: symbol Device:Thermistor_NTC -> pmu_symbols:Thermistor_NTC
