File: bms.kicad_sch (KiCad schematic)
At the start: 71 parts, among them J5 Screw_Terminal_01x02, J6 Molex_Pico-Clasp_1x7_Horizont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, Q10 CSD17579Q5A, Q11 SiA453EDJ, Q12 CSD17579Q5A, Q13 2N7002K, Q5 DMN2056U, Q6 DMN2056U, Q7 DMN2056U, Q8 DMG2301L, Q9 Si1442DH, U1 BQ29410_TSSOP, U2 BQ40Z50RSMT-R2

Commit message: Minimal version without BMS
Parts:
- removed C18, C19, C20, C21, C22, C23, C24, C25, C26, C28, C29, C31, C35: C_100n_16V_X7R_0402, Capacitor_SMD:C_0402_1005Metric, symbol lib:C_Small
- removed C27: TBD, Capacitor_SMD:C_0603_1608Metric, symbol lib:C_Small
- removed C30: C_10n_0402, Capacitor_SMD:C_0402_1005Metric, symbol lib:C_Small
- removed C32: C_2u2_0603, Capacitor_SMD:C_0603_1608Metric, symbol lib:C_Small
- removed C33, C34: C_100n_50V_X7R_0603, Capacitor_SMD:C_0603_1608Metric, symbol lib:C_Small
- removed D5: BAT54J, Diode_SMD:D_SOD-323F, symbol lib:BAT54J
- removed F1: ITV4030L1412NR, ITV4030_LTF, symbol lib:ITV4030L1412NR
- removed J5: Screw_Terminal_01x02, TerminalBlock_Phoenix:TerminalBlock_Phoenix_MKDS-1,5-2_1x02_P5.00mm_Horizontal, symbol lib:Screw_Terminal_01x02
- removed J6: Molex_Pico-Clasp_1x7_Horizontal_SMD_2023960707, Hardware Components Footprints:Molex_Pico-Clasp_1x7_Horizontal_SMD_2023960707, symbol lib:Conn_01x08
- removed PTC1: 10k, Resistor_SMD:R_0402_1005Metric, symbol lib:R_Small
- removed Q10, Q12: CSD17579Q5A, Package_TO_SOT_SMD:TDSON-8-1, symbol lib:CSD17579Q5A
- removed Q11: SiA453EDJ, Package_TO_SOT_SMD:Vishay_PowerPAK_SC70-6L_Single, symbol lib:SiA453EDJ
- removed Q13: 2N7002K, Package_TO_SOT_SMD:SOT-23, symbol lib:2N7002K
- removed Q5, Q6, Q7: DMN2056U, Package_TO_SOT_SMD:SOT-23, symbol lib:DMN2056U
- removed Q8: DMG2301L, Package_TO_SOT_SMD:SOT-23, symbol lib:DMG2301L
- removed Q9: Si1442DH, Package_TO_SOT_SMD:SOT-363_SC-70-6, symbol lib:Si1442DH
- removed R31, R32, R33, R34, R43, R46, R49, R55: R_100R_0402, Resistor_SMD:R_0402_1005Metric, symbol lib:R_Small
- removed R35, R36, R37, R38: R_50R_0402, Resistor_SMD:R_0402_1005Metric, symbol lib:R_Small
- removed R39, R40, R41, R42: R_300R_0402, Resistor_SMD:R_0402_1005Metric, symbol lib:R_Small
- removed R44, R50, R51, R53, R56: R_5k1_0402, Resistor_SMD:R_0402_1005Metric, symbol lib:R_Small
- removed R45: R_51k_0402, Resistor_SMD:R_0402_1005Metric, symbol lib:R_Small
- removed R47: 1mR, Resistor_SMD:R_2010_5025Metric_Pad1.40x2.65mm_HandSolder, symbol lib:R_Small
- removed R48, R54, R57: R_10M_0402, Resistor_SMD:R_0402_1005Metric, symbol lib:R_Small
- removed R52: TBD, Resistor_SMD:R_0603_1608Metric, symbol lib:R_Small
- removed R58, R59: R_10k_0402, Resistor_SMD:R_0402_1005Metric, symbol lib:R_Small
- removed TP1, TP2, TP3, TP4, TP5, TP6, TP7: TP_2.5mm_SMD_1508-0-57-15-00-00-03-0, Hardware Components Footprints:TP_2.5mm_SMD_1508-0-57-15-00-00-03-0, symbol lib:TP_2.5mm_SMD_1508-0-57-15-00-00-03-0
- removed U1: BQ29410_TSSOP, Hardware Components Footprints:TSSOP-8_3x4.4mm_P0.65mm, symbol lib:BQ29410_TSSOP
- removed U2: BQ40Z50RSMT-R2, UserLib:BQ40Z50RSMTR2, symbol lib:BQ40Z50RSMT-R2
- removed xx1: Thermistor_NTC, symbol lib:Thermistor_NTC
Connections:
- no-connect marks 3 -> 0
Other:
- note removed: "ADD TO BOM"
- note removed: "BAT+"
- note removed: "BAT-"
- note removed: "BQ40Z50-R2 Datasheet"
- note removed: "BQ40Z50-R2 product page"
- note removed: "CELL_{1}"
- note removed: "CELL_{2}"
- note removed: "CELL_{3}"
- note removed: "Evaluation module"
- note removed: "External cell balancing"
- note removed: "Fast Cell Balancing Using External MOSFET app note"
- note removed: "I_{precharge} = (V_{CHARGER} - V_{BAT}))/R_{1}"
- note removed: "REFERENCES"
- note removed: "When not using external balancing replace R[11..13] with 100Ohm and depopulate R14,26,28,29 Q5 Q12 Q8 Q10"
- note removed: "t_{d} = [1.2V * C_{Delay}]/ 0.18u"
- title: Robot power supply -> (none)
