File: robot-pmu-hw.kicad_pcb (KiCad board)
At the start: 2 copper layers, 33.2 x 39.2 mm, 62 parts, among them J2 Molex_Pico-Clasp_1x7_Horizont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, J3 Screw_Terminal_01x02, Q13 DMG2301L, Q14 Si1442DH, Q15 CSD17579Q5A, Q16 SiA453EDJ, Q18 2N7002K, Q2 CSD17579Q5A, Q5 DMN2056U, Q8 DMN2056U, Q9 DMN2056U, U1 BQ29410_TSSOP, U4 BQ40Z50RSMT-R2

Commit message: Link footprints and symbols to local lib
Parts:
- C10, C11, C12, C14, C15, C19, C2, C24, C3, C31, C32, C4, C6, C9: footprint Capacitor_SMD:C_0402_1005Metric -> pmu_footprint:C_0402_1005Metric
- C28, C33, C34, C8: footprint Capacitor_SMD:C_0603_1608Metric -> pmu_footprint:C_0603_1608Metric
- D1: footprint Diode_SMD:D_SOD-323F -> pmu_footprint:D_SOD-323F
- J2: footprint Hardware Components Footprints:Molex_Pico-Clasp_1x7_Horizontal_SMD_2023960707 -> pmu_footprint:Molex_Pico-Clasp_1x7_Horizontal_SMD_2023960707
- J3: footprint TerminalBlock_Phoenix:TerminalBlock_Phoenix_MKDS-1,5-2_1x02_P5.00mm_Horizontal -> pmu_footprint:TerminalBlock_Phoenix_MKDS-1,5-2_1x02_P5.00mm_Horizontal
- PTC2, R10, R12, R13, R14, R16, R17, R18, R19, R2, R20, R23, R26, R28, R29, R3, R30, R33, R37, R4, R42, R43, R44, R46, R5, R56, R6, R9: footprint Resistor_SMD:R_0402_1005Metric -> pmu_footprint:R_0402_1005Metric
- Q13, Q18, Q5, Q8, Q9: footprint Package_TO_SOT_SMD:SOT-23 -> pmu_footprint:SOT-23
- Q14: footprint Package_TO_SOT_SMD:SOT-363_SC-70-6 -> pmu_footprint:SOT-363_SC-70-6
- Q15, Q2: footprint Package_TO_SOT_SMD:TDSON-8-1 -> pmu_footprint:TDSON-8-1
- Q16: footprint Package_TO_SOT_SMD:Vishay_PowerPAK_SC70-6L_Single -> pmu_footprint:Vishay_PowerPAK_SC70-6L_Single
- R45: footprint Resistor_SMD:R_2010_5025Metric_Pad1.40x2.65mm_HandSolder -> pmu_footprint:R_2010_5025Metric_Pad1.40x2.65mm_HandSolder
- R50: footprint Resistor_SMD:R_0603_1608Metric -> pmu_footprint:R_0603_1608Metric
- U1: footprint Hardware Components Footprints:TSSOP-8_3x4.4mm_P0.65mm -> pmu_footprint:TSSOP-8_3x4.4mm_P0.65mm
- U4: footprint UserLib:BQ40Z50RSMTR2 -> pmu_footprint:BQ40Z50RSMTR2
Changed lines of the file:
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@@
 	(net 56 "/bms/~{PRES_OR_}SHUTDN")
 	(net 57 "/bms/SMBC")
-	(footprint "Resistor_SMD:R_0402_1005Metric"
+	(footprint "pmu_footprint:R_0402_1005Metric"
 		(layer "F.Cu")
 		(at 131.535 77.85)
@@
 		)
 	)
-	(footprint "Resistor_SMD:R_2010_5025Metric_Pad1.40x2.65mm_HandSolder"
+	(footprint "pmu_footprint:R_2010_5025Metric_Pad1.40x2.65mm_HandSolder"
 		(layer "F.Cu")
 		(at 142.685 109.05)
@@
 		)
 	)
-	(footprint "Resistor_SMD:R_0402_1005Metric"
+	(footprint "pmu_footprint:R_0402_1005Metric"
 		(layer "F.Cu")
 		(at 134.445 91.78)
@@
 		)
 	)
-	(footprint "Package_TO_SOT_SMD:Vishay_PowerPAK_SC70-6L_Single"
+	(footprint "pmu_footprint:Vishay_PowerPAK_SC70-6L_Single"
 		(layer "F.Cu")
 		(at 153.86 103.425)
@@
 		)
 	)
-	(footprint "Resistor_SMD:R_0402_1005Metric"
+	(footprint "pmu_footprint:R_0402_1005Metric"
 		(layer "F.Cu")
 		(at 131.535 79.84)
@@
 		)
 	)
-	(footprint "Resistor_SMD:R_0402_1005Metric"
+	(footprint "pmu_footprint:R_0402_1005Metric"
 		(layer "F.Cu")
 		(at 134.445 77.85)
@@
 		)
 	)
-	(footprint "Package_TO_SOT_SMD:SOT-23"
+	(footprint "pmu_footprint:SOT-23"
 		(layer "F.Cu")
 		(at 149.475 104.55)
@@
 		)
 	)
-	(footprint "Resistor_SMD:R_0402_1005Metric"
+	(footprint "pmu_footprint:R_0402_1005Metric"
 		(layer "F.Cu")
 		(at 131.535 83.82)
@@
 		)
 	)
-	(footprint "Capacitor_SMD:C_0402_1005Metric"
+	(footprint "pmu_footprint:C_0402_1005Metric"
 		(layer "F.Cu")
 		(at 131.475 109.49)
@@
 		)
 	)
-	(footprint "Capacitor_SMD:C_0402_1005Metric"
+	(footprint "pmu_footprint:C_0402_1005Metric"
 		(layer "F.Cu")
 		(at 131.475 101.61)
@@
 		)
 	)
-	(footprint "Resistor_SMD:R_0603_1608Metric"
+	(footprint "pmu_footprint:R_0603_1608Metric"
 		(layer "F.Cu")
 		(at 153.935 100.27)
@@
 		)
 	)
-	(footprint "Capacitor_SMD:C_0402_1005Metric"
+	(footprint "pmu_footprint:C_0402_1005Metric"
 		(layer "F.Cu")
 		(at 134.345 105.55)
@@
 		)
 	)
-	(footprint "Capacitor_SMD:C_0402_1005Metric"
+	(footprint "pmu_footprint:C_0402_1005Metric"
 		(layer "F.Cu")
 		(at 128.605 105.55)
@@
 		)
 	)
-	(footprint "Capacitor_SMD:C_0603_1608Metric"
+	(footprint "pmu_footprint:C_0603_1608Metric"
 		(layer "F.Cu")
 		(at 153.935 92.74)
@@
 		)
 	)
-	(footprint "Capacitor_SMD:C_0402_1005Metric"
+	(footprint "pmu_footprint:C_0402_1005Metric"
 		(layer "F.Cu")
 		(at 128.605 101.61)
@@
 		)
 	)
-	(footprint "Package_TO_SOT_SMD:SOT-23"
+	(footprint "pmu_footprint:SOT-23"
 		(layer "F.Cu")
 		(at 149.475 91.2)
@@
 		)
 	)
-	(footprint "Capacitor_SMD:C_0402_1005Metric"
+	(footprint "pmu_footprint:C_0402_1005Metric"
 		(layer "F.Cu")
 		(at 134.345 107.52)
@@
 		)
 	)
-	(footprint "Capacitor_SMD:C_0402_1005Metric"
+	(footprint "pmu_footprint:C_0402_1005Metric"
 		(layer "F.Cu")
 		(at 128.605 109.49)
@@
 		)
 	)
-	(footprint "Resistor_SMD:R_0402_1005Metric"
+	(footprint "pmu_footprint:R_0402_1005Metric"
 		(layer "F.Cu")
 		(at 137.355 81.83)
@@
 		)
 	)
-	(footprint "Capacitor_SMD:C_0603_1608Metric"
+	(footprint "pmu_footprint:C_0603_1608Metric"
 		(layer "F.Cu")
 		(at 153.935 95.25)
@@
 		)
 	)
-	(footprint "Hardware Components Footprints:Molex_Pico-Clasp_1x7_Horizontal_SMD_2023960707"
+	(footprint "pmu_footprint:Molex_Pico-Clasp_1x7_Horizontal_SMD_2023960707"
 		(layer "F.Cu")
 		(at 132.795 97)
@@
 		)
 	)
-	(footprint "Resistor_SMD:R_0402_1005Metric"
+	(footprint "pmu_footprint:R_0402_1005Metric"
 		(layer "F.Cu")
 		(at 128.625 89.79)
@@
 		)
 	)
-	(footprint "Resistor_SMD:R_0402_1005Metric"
+	(footprint "pmu_footprint:R_0402_1005Metric"
 		(layer "F.Cu")
 		(at 131.535 81.83)
@@
 		)
 	)
-	(footprint "Capacitor_SMD:C_0402_1005Metric"
+	(footprint "pmu_footprint:C_0402_1005Metric"
 		(layer "F.Cu")
 		(at 134.345 101.61)
@@
 		)
 	)
-	(footprint "Resistor_SMD:R_0402_1005Metric"
+	(footprint "pmu_footprint:R_0402_1005Metric"
 		(layer "F.Cu")
 		(at 131.535 85.81)
@@
 		)
 	)
-	(footprint "Capacitor_SMD:C_0603_1608Metric"
+	(footprint "pmu_footprint:C_0603_1608Metric"
 		(layer "F.Cu")
 		(at 153.935 97.76)
@@
 		)
 	)
-	(footprint "Capacitor_SMD:C_0402_1005Metric"
+	(footprint "pmu_footprint:C_0402_1005Metric"
 		(layer "F.Cu")
 		(at 134.345 103.58)
@@
 		)
 	)
-	(footprint "Capacitor_SMD:C_0402_1005Metric"
+	(footprint "pmu_footprint:C_0402_1005Metric"
 		(layer "F.Cu")
 		(at 131.475 107.52)
@@
 		)
 	)
-	(footprint "Resistor_SMD:R_0402_1005Metric"
+	(footprint "pmu_footprint:R_0402_1005Metric"
 		(layer "F.Cu")
 		(at 134.445 87.8)
@@
 		)
 	)
-	(footprint "Resistor_SMD:R_0402_1005Metric"
+	(footprint "pmu_footprint:R_0402_1005Metric"
 		(layer "F.Cu")
 		(at 128.625 91.78)
@@
 		)
 	)
-	(footprint "Resistor_SMD:R_0402_1005Metric"
+	(footprint "pmu_footprint:R_0402_1005Metric"
 		(layer "F.Cu")
 		(at 134.445 79.84)
@@
 		)
 	)
-	(footprint "TerminalBlock_Phoenix:TerminalBlock_Phoenix_MKDS-1,5-2_1x02_P5.00mm_Horizontal"
+	(footprint "pmu_footprint:TerminalBlock_Phoenix_MKDS-1,5-2_1x02_P5.00mm_Horizontal"
 		(layer "F.Cu")
 		(at 142.335 83.09)
@@
 		)
 	)
-	(footprint "Resistor_SMD:R_0402_1005Metric"
+	(footprint "pmu_footprint:R_0402_1005Metric"
 		(layer "F.Cu")
 		(at 134.445 83.82)
@@
 		)
 	)
-	(footprint "UserLib:BQ40Z50RSMTR2"
+	(footprint "pmu_footprint:BQ40Z50RSMTR2"
 		(layer "F.Cu")
 		(at 154.26 79.705)
@@
 		)
 	)
-	(footprint "Package_TO_SOT_SMD:TDSON-8-1"
+	(footprint "pmu_footprint:TDSON-8-1"
 		(layer "F.Cu")
 		(at 142.915 99.04)
@@
 		)
 	)
-	(footprint "Resistor_SMD:R_0402_1005Metric"
+	(footprint "pmu_footprint:R_0402_1005Metric"
 		(layer "F.Cu")
 		(at 131.535 91.78)
@@
 		)
 	)
-	(footprint "Hardware Components Footprints:TSSOP-8_3x4.4mm_P0.65mm"
+	(footprint "pmu_footprint:TSSOP-8_3x4.4mm_P0.65mm"
 		(layer "F.Cu")
 		(at 142.785 104.67)
@@
 		)
 	)
-	(footprint "Resistor_SMD:R_0402_1005Metric"
+	(footprint "pmu_footprint:R_0402_1005Metric"
 		(layer "F.Cu")
 		(at 131.535 89.79)
@@
 		)
 	)
-	(footprint "Package_TO_SOT_SMD:SOT-23"
+	(footprint "pmu_footprint:SOT-23"
 		(layer "F.Cu")
 		(at 149.475 95.65)
@@
 		)
 	)
-	(footprint "Capacitor_SMD:C_0402_1005Metric"
+	(footprint "pmu_footprint:C_0402_1005Metric"
 		(layer "F.Cu")
 		(at 128.605 107.52)
@@
 		)
 	)
-	(footprint "Resistor_SMD:R_0402_1005Metric"
+	(footprint "pmu_footprint:R_0402_1005Metric"
 		(layer "F.Cu")
 		(at 128.625 85.81)
@@
 		)
 	)
-	(footprint "Resistor_SMD:R_0402_1005Metric"
+	(footprint "pmu_footprint:R_0402_1005Metric"
 		(layer "F.Cu")
 		(at 128.625 79.84)
@@
 		)
 	)
-	(footprint "Resistor_SMD:R_0402_1005Metric"
+	(footprint "pmu_footprint:R_0402_1005Metric"
 		(layer "F.Cu")
 		(at 131.535 87.8)
@@
 		)
 	)
-	(footprint "Resistor_SMD:R_0402_1005Metric"
+	(footprint "pmu_footprint:R_0402_1005Metric"
 		(layer "F.Cu")
 		(at 128.625 81.83)
@@
 		)
 	)
-	(footprint "Capacitor_SMD:C_0402_1005Metric"
+	(footprint "pmu_footprint:C_0402_1005Metric"
 		(layer "F.Cu")
 		(at 131.475 103.58)
@@
 		)
 	)
-	(footprint "Diode_SMD:D_SOD-323F"
+	(footprint "pmu_footprint:D_SOD-323F"
 		(layer "F.Cu")
 		(at 154.1 106.7)
@@
 		)
 	)
-	(footprint "Resistor_SMD:R_0402_1005Metric"
+	(footprint "pmu_footprint:R_0402_1005Metric"
 		(layer "F.Cu")
 		(at 134.445 85.81)
@@
 		)
 	)
-	(footprint "Resistor_SMD:R_0402_1005Metric"
+	(footprint "pmu_footprint:R_0402_1005Metric"
 		(layer "F.Cu")
 		(at 134.445 81.83)
@@
 		)
 	)
-	(footprint "Package_TO_SOT_SMD:SOT-363_SC-70-6"
+	(footprint "pmu_footprint:SOT-363_SC-70-6"
 		(layer "F.Cu")
 		(at 152.985 84.555)
@@
 		)
 	)
-	(footprint "Resistor_SMD:R_0402_1005Metric"
+	(footprint "pmu_footprint:R_0402_1005Metric"
 		(layer "F.Cu")
 		(at 128.625 83.82)
@@
 		)
 	)
-	(footprint "Package_TO_SOT_SMD:TDSON-8-1"
+	(footprint "pmu_footprint:TDSON-8-1"
 		(layer "F.Cu")
 		(at 142.915 92.33)
@@
 		)
 	)
-	(footprint "Capacitor_SMD:C_0402_1005Metric"
+	(footprint "pmu_footprint:C_0402_1005Metric"
 		(layer "F.Cu")
 		(at 131.475 105.55)
@@
 		)
 	)
-	(footprint "Resistor_SMD:R_0402_1005Metric"
+	(footprint "pmu_footprint:R_0402_1005Metric"
 		(layer "F.Cu")
 		(at 137.355 77.85)
@@
 		)
 	)
-	(footprint "Resistor_SMD:R_0402_1005Metric"
+	(footprint "pmu_footprint:R_0402_1005Metric"
 		(layer "F.Cu")
 		(at 134.445 89.79)
@@
 		)
 	)
-	(footprint "Package_TO_SOT_SMD:SOT-23"
+	(footprint "pmu_footprint:SOT-23"
 		(layer "F.Cu")
 		(at 149.475 100.1)
@@
 		)
 	)
-	(footprint "Capacitor_SMD:C_0603_1608Metric"
+	(footprint "pmu_footprint:C_0603_1608Metric"
 		(layer "F.Cu")
 		(at 153.935 90.23)
@@
 		)
 	)
-	(footprint "Resistor_SMD:R_0402_1005Metric"
+	(footprint "pmu_footprint:R_0402_1005Metric"
 		(layer "F.Cu")
 		(at 128.625 77.85)
@@
 		)
 	)
-	(footprint "Resistor_SMD:R_0402_1005Metric"
+	(footprint "pmu_footprint:R_0402_1005Metric"
 		(layer "F.Cu")
 		(at 137.355 83.82)
@@
 		)
 	)
-	(footprint "Resistor_SMD:R_0402_1005Metric"
+	(footprint "pmu_footprint:R_0402_1005Metric"
 		(layer "F.Cu")
 		(at 128.625 87.8)
@@
 		)
 	)
-	(footprint "Capacitor_SMD:C_0402_1005Metric"
+	(footprint "pmu_footprint:C_0402_1005Metric"
 		(layer "F.Cu")
 		(at 128.605 103.58)
@@
 		)
 	)
-	(footprint "Package_TO_SOT_SMD:SOT-23"
+	(footprint "pmu_footprint:SOT-23"
 		(layer "F.Cu")
 		(at 149.475 109)
@@
 		)
 	)
-	(footprint "Resistor_SMD:R_0402_1005Metric"
+	(footprint "pmu_footprint:R_0402_1005Metric"
 		(layer "F.Cu")
 		(at 137.355 79.84)
