File: channel_output_0.kicad_sch (KiCad schematic)
At the start: 27 parts, among them IC7 TPS56637RPAR, J12 Conn_01x02, Q7 2N7002_SOT-23-3, U5 MCP4725xxx-xCH

Commit message: test points
Parts:
- added TP1, TP13, TP17, TP19, TP22, TP26, TP5, TP9: TP_2.54mm_THT_5002, Hardware Components Footprints:TP_2.54mm_THT_Keystone_500x, symbol Hardware Components:TP_2.54mm_THT_5002
Connections:
- net +16V: now also TP9.1
- net CH_ADC: now also TP13.1
- net GND: now also TP22.1, TP26.1
- net at IC7.1 (EN), R51.2, R52.2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: now also TP17.1
- net at C53.1, IC7.2 (FB), R55.1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: now also TP5.1
- net at C54.2, C55.2, C56.2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: now also TP1.1
- net at C52.2, IC7.6 (SW), L5.1: now also TP19.1
